Commit message: Update materials and colors in robot_core.xacro

File: description/robot_core.xacro (robot description, xacro)
@@ -13,4 +13,7 @@
     <material name="black">
         <color rgba="0 0 0 1"/>
+    </material>
+<material name="red">
+        <color rgba="1 0 0 1"/>
     </material>
     <link name="base_link">
@@ -34,5 +37,4 @@
         <box size="0.3 0.3 0.15"/>
       </geometry>
-      <material name="white"/>
     </collision>
     <!-- Inertial from macro -->
@@ -41,5 +43,5 @@
     </xacro:inertial_box>
     <gazebo reference="chassis">
-    <material>Gazebo/White</material>
+    <material>Gazebo/Orange</material>
     </gazebo>
   </link>
@@ -62,5 +64,4 @@
         <cylinder length="0.04" radius="0.05" />
       </geometry>
-      <material name="blue"/>
     </collision>
     <!-- Inertial from macro -->
@@ -69,5 +70,5 @@
     </xacro:inertial_cylinder>
     <gazebo reference="left_wheel">
-    <material>Gazebo/blue</material>
+    <material>Gazebo/Blue</material>
     </gazebo>
   </link>
@@ -90,5 +91,4 @@
         <cylinder length="0.04" radius="0.05" />
       </geometry>
-      <material name="blue"/>
     </collision>
     <!-- Inertial from macro -->
@@ -97,5 +97,5 @@
     </xacro:inertial_cylinder>
     <gazebo reference="right_wheel">
-        <material>Gazebo/blue</material>
+        <material>Gazebo/Blue</material>
     </gazebo>
   </link>
@@ -116,5 +116,4 @@
         <geometry>
          <sphere radius="0.05" />
-         <material name="black"/>
         </geometry>
     </collision>
